Commit message: Add controller

File: pudu_description/urdf/components/wheels/wheel.urdf.xacro (robot description, xacro)
@@ -3,5 +3,5 @@
     <xacro:property name="wheel_radius" value="0.1"/>
     <xacro:property name="wheel_length" value="0.05"/>
-    <xacro:property name="wheel_mass" value="3.0"/>
+    <xacro:property name="wheel_mass" value="1.0"/>
     <xacro:macro name="wheel" params="prefix parent *origin">
         <joint name="${prefix}_wheel_joint" type="continuous">

File: pudu_description/urdf/robots/pudu.urdf.xacro (robot description, xacro)
@@ -5,17 +5,31 @@
     <xacro:include filename="$(find pudu_description)/urdf/components/base/base.urdf.xacro" />
     <xacro:include filename="$(find pudu_description)/urdf/components/wheels/wheel.urdf.xacro" />
-    <xacro:include filename="$(find pudu_description)/urdf/components/wheels/steering_wheel.urdf.xacro" />
+    <xacro:include filename="$(find pudu_description)/urdf/components/plugins/control.urdf.xacro" />
+    <xacro:include filename="$(find pudu_description)/urdf/components/plugins/transmission.urdf.xacro" />
+    <xacro:include filename="$(find pudu_description)/urdf/components/plugins/gz_control.urdf.xacro" />
     <xacro:base />
-    <xacro:steering_wheel prefix="front" parent="base_link">
-        <origin xyz="-0.3 0 -0.35" rpy="0 0 0"/>
-    </xacro:steering_wheel>
-    <xacro:steering_wheel prefix="rear" parent="base_link">
-        <origin xyz="0.3 0 -0.35" rpy="0 0 0"/>
-    </xacro:steering_wheel>
-    <xacro:wheel prefix="left" parent="base_link">
-        <origin xyz="0 -0.25 -0.3" rpy="0 0 0"/>
+    <xacro:property name="wheel_x" value="${base_length/2 - 0.08}"/>
+    <xacro:property name="wheel_y" value="${base_width/2 - 0.08}"/>
+    <xacro:property name="wheel_z" value="${-base_height/2 - clearance + wheel_radius}"/>
+    <xacro:wheel prefix="front_left" parent="base_link">
+        <origin xyz="${wheel_x} ${wheel_y} ${wheel_z}" rpy="0 0 -0.785398"/>
     </xacro:wheel>
-    <xacro:wheel prefix="right" parent="base_link">
-        <origin xyz="0 0.25 -0.3" rpy="0 0 0"/>
+    <xacro:wheel prefix="rear_left" parent="base_link">
+        <origin xyz="-${wheel_x} ${wheel_y} ${wheel_z}" rpy="0 0 0.785398"/>
     </xacro:wheel>
+    <xacro:wheel prefix="rear_right" parent="base_link">
+        <origin xyz="-${wheel_x} -${wheel_y} ${wheel_z}" rpy="0 0 2.35617"/>
+    </xacro:wheel>
+    <xacro:wheel prefix="front_right" parent="base_link">
+        <origin xyz="${wheel_x} -${wheel_y} ${wheel_z}" rpy="0 0 -2.35617"/>
+    </xacro:wheel>
+     <xacro:control>
+        <transmissions>
+            <xacro:transmission joint="front_left_wheel_joint"/>
+            <xacro:transmission joint="front_right_wheel_joint"/>
+            <xacro:transmission joint="rear_left_wheel_joint"/>
+            <xacro:transmission joint="rear_right_wheel_joint"/>
+        </transmissions>
+    </xacro:control>
+    <xacro:gz_control namespace="$(arg robot_namespace)"/>
 </robot>
