Commit message: Add visualization and lidar

File: pudu_description/urdf/components/base/base.urdf.xacro (robot description, xacro)
@@ -13,11 +13,11 @@
         <link name="base_link">
             <visual>
-                <origin xyz="0 0 0" rpy="0.0 0.0 0.0" />
+                <origin xyz="0 0 -0.37" rpy="0.0 0.0 ${pi/2}" />
                 <geometry>
-                    <box size="${base_length} ${base_width} ${base_height}"/>
+                    <mesh filename="file://$(find pudu_description)/meshes/base/base.dae" scale="${base_length} ${base_width} ${base_height}"/>
                 </geometry>
             </visual>
             <collision>
-                <origin xyz="0 0 0" rpy="0.0 0.0 0.0" />
+                <origin xyz="0 0 -0.37" rpy="0.0 0.0 0.0" />
                 <geometry>
                     <box size="${base_length} ${base_width} ${base_height}"/>

File: pudu_description/urdf/robots/pudu.urdf.xacro (robot description, xacro)
@@ -8,4 +8,5 @@
     <xacro:include filename="$(find pudu_description)/urdf/components/plugins/transmission.urdf.xacro" />
     <xacro:include filename="$(find pudu_description)/urdf/components/plugins/gz_control.urdf.xacro" />
+    <xacro:include filename="$(find pudu_description)/urdf/components/sensors/lidar.urdf.xacro" />
     <xacro:base />
     <xacro:property name="wheel_x" value="${base_length/2 - 0.08}"/>
@@ -33,3 +34,6 @@
     </xacro:control>
     <xacro:gz_control namespace="$(arg robot_namespace)"/>
+    <xacro:lidar prefix="lidar" parent="base_link" ns="$(arg robot_namespace)">
+        <origin xyz="0.25 0.0 2.9" rpy="0.0 0.0 0.0"/>
+    </xacro:lidar>
 </robot>

Commit message: Fix meshes and lidar

File: pudu_description/urdf/components/base/base.urdf.xacro (robot description, xacro)
@@ -1,7 +1,7 @@
 <?xml version="1.0"?>
 <robot xmlns:xacro="http://ros.org/wiki/xacro">
-    <xacro:property name="base_length" value="0.663"/>
-    <xacro:property name="base_width" value="0.568"/>
-    <xacro:property name="base_height" value="0.682"/>
+    <xacro:property name="base_length" value="0.6"/>
+    <xacro:property name="base_width" value="0.6"/>
+    <xacro:property name="base_height" value="0.9"/>
     <xacro:property name="clearance" value="0.05"/>
     <xacro:property name="mass" value="60.0"/>
@@ -13,11 +13,11 @@
         <link name="base_link">
             <visual>
-                <origin xyz="0 0 -0.37" rpy="0.0 0.0 ${pi/2}" />
+                <origin xyz="0 0 -0.59" rpy="0.0 0.0 ${pi/2}" />
                 <geometry>
-                    <mesh filename="file://$(find pudu_description)/meshes/base/base.dae" scale="${base_length} ${base_width} ${base_height}"/>
+                    <mesh filename="file://$(find pudu_description)/meshes/base/base.dae" scale="0.4 0.4 0.2"/>
                 </geometry>
             </visual>
             <collision>
-                <origin xyz="0 0 -0.37" rpy="0.0 0.0 0.0" />
+                <origin xyz="0 0 0" rpy="0.0 0.0 0.0" />
                 <geometry>
                     <box size="${base_length} ${base_width} ${base_height}"/>

File: pudu_description/urdf/components/sensors/lidar.urdf.xacro (robot description, xacro)
@@ -10,5 +10,5 @@
     <link name="${prefix}_link">
       <visual>
-        <origin xyz="-0.25 0 0.35" rpy="0 0 0"/>
+        <origin xyz="0 0 0" rpy="0 0 0"/>
         <geometry>
             <mesh filename="file://$(find pudu_description)/meshes/sensors/hokuyo_urg_04lx_ug01.stl"/>
@@ -16,5 +16,5 @@
       </visual>
       <collision>
-			  <origin xyz="-0.25 0 0.35" rpy="0 0 0"/>
+			  <origin xyz="0 0 0" rpy="0 0 0"/>
 			  <geometry>
 				  <mesh filename="file://$(find pudu_description)/meshes/sensors/hokuyo_urg_04lx_ug01.stl"/>

File: pudu_description/urdf/robots/pudu.urdf.xacro (robot description, xacro)
@@ -35,5 +35,5 @@
     <xacro:gz_control namespace="$(arg robot_namespace)"/>
     <xacro:lidar prefix="lidar" parent="base_link" ns="$(arg robot_namespace)">
-        <origin xyz="0.25 0.0 2.9" rpy="0.0 0.0 0.0"/>
+        <origin xyz="0.0 0.0 0.5" rpy="0.0 0.0 0.0"/>
     </xacro:lidar>
 </robot>
